File: ATTAMI.sch (EAGLE design)
At the start: 19 parts, among them J1 CON_HEADER_1X02-PTH, J2 MICRO-USB_ALIEXPRESS, J3 CON_HEADER_1X02-PTH, U1 MIC5225, U2 ATTINY85

Commit message: 15b-03
Parts:
- J4: value (none) -> CON_HEADER_1X06-PTH; device adafruit:PINHD-1X6CB -> dp_devices:CON_HEADER_1X06-PTH
Other:
- note added: "AT TAMI Ver. 15b03"
- note removed: "AT TAMI Ver. 15b"
Changed lines of the file:
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@@
 <part name="GND4" library="SparkFun" deviceset="GND" device=""/>
 <part name="U$2" library="microbuilder" deviceset="MOUNTINGHOLE" device="2.0" value="MOUNTINGHOLE2.0"/>
-<part name="J4" library="adafruit" deviceset="PINHD-1X6" device="CB"/>
 <part name="J1" library="dp_devices" deviceset="CON_HEADER_1X02" device="-PTH"/>
 <part name="J3" library="dp_devices" deviceset="CON_HEADER_1X02" device="-PTH"/>
+<part name="J4" library="dp_devices" deviceset="CON_HEADER_1X06" device="-PTH"/>
 </parts>
 <sheets>
@@
 <text x="205.74" y="0" size="2.54" layer="100" font="vector">T.A.M.I hackerspace crew
 LICENSE: CERN OHL 1.7</text>
-<text x="205.74" y="-7.62" size="2.54" layer="100" font="vector">AT TAMI Ver. 15b</text>
+<text x="205.74" y="-7.62" size="2.54" layer="100" font="vector">AT TAMI Ver. 15b03</text>
 <text x="205.74" y="-15.24" size="2.54" layer="100" font="vector">&gt;LAST_DATE_TIME</text>
 <wire x1="198.12" y1="-20.32" x2="198.12" y2="17.78" width="0.254" layer="100"/>
@@
 <instance part="GND4" gate="1" x="58.42" y="93.98"/>
 <instance part="U$2" gate="G$1" x="142.24" y="162.56"/>
-<instance part="J4" gate="A" x="215.9" y="137.16"/>
 <instance part="J1" gate="J" x="33.02" y="144.78" rot="MR0"/>
 <instance part="J3" gate="J" x="83.82" y="162.56" rot="MR0"/>
+<instance part="J4" gate="G$1" x="215.9" y="139.7"/>
 </instances>
 <busses>
@@
 <wire x1="170.18" y1="137.16" x2="175.26" y2="137.16" width="0.1524" layer="91"/>
 <wire x1="175.26" y1="137.16" x2="175.26" y2="106.68" width="0.1524" layer="91"/>
-<wire x1="175.26" y1="137.16" x2="213.36" y2="137.16" width="0.1524" layer="91"/>
+<wire x1="175.26" y1="137.16" x2="215.9" y2="137.16" width="0.1524" layer="91"/>
 <junction x="175.26" y="137.16"/>
-<pinref part="J4" gate="A" pin="4"/>
+<pinref part="J4" gate="G$1" pin="4"/>
 </segment>
 </net>
@@
 <segment>
 <pinref part="U2" gate="G$1" pin="PB0(MOSI)"/>
-<wire x1="213.36" y1="144.78" x2="170.18" y2="144.78" width="0.1524" layer="91"/>
-<pinref part="J4" gate="A" pin="1"/>
+<wire x1="215.9" y1="144.78" x2="170.18" y2="144.78" width="0.1524" layer="91"/>
+<pinref part="J4" gate="G$1" pin="1"/>
 </segment>
 </net>
@@
 <segment>
 <pinref part="U2" gate="G$1" pin="PB2(SCK/ADC1)"/>
-<wire x1="213.36" y1="139.7" x2="170.18" y2="139.7" width="0.1524" layer="91"/>
-<pinref part="J4" gate="A" pin="3"/>
+<wire x1="215.9" y1="139.7" x2="170.18" y2="139.7" width="0.1524" layer="91"/>
+<pinref part="J4" gate="G$1" pin="3"/>
 </segment>
 </net>
@@
 <wire x1="170.18" y1="134.62" x2="180.34" y2="134.62" width="0.1524" layer="91"/>
 <wire x1="180.34" y1="134.62" x2="180.34" y2="104.14" width="0.1524" layer="91"/>
-<wire x1="180.34" y1="134.62" x2="213.36" y2="134.62" width="0.1524" layer="91"/>
+<wire x1="180.34" y1="134.62" x2="215.9" y2="134.62" width="0.1524" layer="91"/>
 <junction x="180.34" y="134.62"/>
-<pinref part="J4" gate="A" pin="5"/>
+<pinref part="J4" gate="G$1" pin="5"/>
 </segment>
 </net>
@@
 <wire x1="170.18" y1="132.08" x2="190.5" y2="132.08" width="0.1524" layer="91"/>
 <pinref part="S1" gate="G$1" pin="2"/>
-<wire x1="190.5" y1="132.08" x2="213.36" y2="132.08" width="0.1524" layer="91"/>
+<wire x1="190.5" y1="132.08" x2="215.9" y2="132.08" width="0.1524" layer="91"/>
 <junction x="190.5" y="132.08"/>
-<pinref part="J4" gate="A" pin="6"/>
+<pinref part="J4" gate="G$1" pin="6"/>
 </segment>
 </net>
@@
 <segment>
 <pinref part="U2" gate="G$1" pin="PB1(MISO)"/>
-<wire x1="213.36" y1="142.24" x2="170.18" y2="142.24" width="0.1524" layer="91"/>
-<pinref part="J4" gate="A" pin="2"/>
-</segment>
-</net>
+<wire x1="215.9" y1="142.24" x2="170.18" y2="142.24" width="0.1524" layer="91"/>
+<pinref part="J4" gate="G$1" pin="2"/>
+</segment>
+</net>

Commit message: ver 16
now with stock DOC_frame
Other:
- note removed: "AT TAMI Ver. 15b03"
Changed lines of the file:
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@@
 <?xml version="1.0" encoding="utf-8"?>
 <!DOCTYPE eagle SYSTEM "eagle.dtd">
-<eagle version="6.6.0">
+<eagle version="6.3">
 <drawing>
 <settings>
@@
 <part name="J3" library="dp_devices" deviceset="CON_HEADER_1X02" device="-PTH"/>
 <part name="J4" library="dp_devices" deviceset="CON_HEADER_1X06" device="-PTH"/>
+<part name="FRAME1" library="frames" deviceset="A4L-LOC" device=""/>
 </parts>
 <sheets>
@@
 <vertex x="0.3796875" y="-0.91665"/>
 </polygon>
-<frame x1="-2.54" y1="-25.4" x2="266.7" y2="185.42" columns="8" rows="5" layer="100"/>
-<text x="205.74" y="0" size="2.54" layer="100" font="vector">T.A.M.I hackerspace crew
+<text x="165.1" y="12.7" size="2.54" layer="100" font="vector">T.A.M.I hackerspace crew
 LICENSE: CERN OHL 1.7</text>
-<text x="205.74" y="-7.62" size="2.54" layer="100" font="vector">AT TAMI Ver. 15b03</text>
-<text x="205.74" y="-15.24" size="2.54" layer="100" font="vector">&gt;LAST_DATE_TIME</text>
-<wire x1="198.12" y1="-20.32" x2="198.12" y2="17.78" width="0.254" layer="100"/>
-<wire x1="198.12" y1="17.78" x2="261.62" y2="17.78" width="0.254" layer="100"/>
 </plain>
 <instances>
@@
 <instance part="J3" gate="J" x="83.82" y="162.56" rot="MR0"/>
 <instance part="J4" gate="G$1" x="215.9" y="139.7"/>
+<instance part="FRAME1" gate="G$1" x="0" y="0"/>
 </instances>
 <busses>
