File: ATTAMI.sch (EAGLE design)
At the start: 23 parts, among them U1 MIC5225, U2 ATTINY85

Commit message: seocnd batch to fab
zv additions
Added + and gnd marking near the coin-cell legs on bottom side of the
PCB.
Made some legend changing on the schematic.
Parts:
- removed COIN_CELL, COIN_CELL_GND: (no value), adafruit:PINHD-1X1CB
- added COIN_CELL_(+), COIN_CELL_(-): (no value), adafruit:PINHD-1X1CB
Connections:
- net GND: now also COIN_CELL_(-).1; no longer COIN_CELL_GND.1
- net N$4: now also COIN_CELL_(+).1; no longer COIN_CELL.1
Other:
- note added: "Notes: 1. D1 and D2 are Blue LEDs they might not light when using Vi_BAT <4V~ 2. When VCC is less than 5V change the system clock of the ATTINY85 to 8MHz or less (refer to the datasheet P163 Section 21-3 Speed)"
- note added: "Reset"
- note added: "VCC (output)"
- note added: "V_BAT (input)"
- note removed: "Notes: 1. D2 and D3 are Blue LEDs they might not light when using Vi_BAT <4V~ 2. When VCC is less than 5V change the system clock of the ATTINY85 to 8MHz or less (refer to datasheet of P163 speed figure 21-1)"
- moved on the sheet: C1, C2, D1, D2, D3, D4, D5, J1, J2, J3, R1, R2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
