File: ATTAMI-V0.00.sch (EAGLE design)
At the start: 25 parts, among them U1 MIC5225, U2 ATTINY85-20SU

Commit message: hl version
Parts:
- 1117: device ATtami:XXX1117-SOT89 -> ATtami:XXX1117
- SJ1: value (none) -> JUMPER-PAD-2-NC_BY_TRACE; device ATtami:SOLDERJUMPERCLOSED -> SparkFun-Passives:JUMPER-PAD-2-NC_BY_TRACE
- SJ2: value (none) -> JUMPER-PAD-3-2OF3_NC_BY_TRACE_SMALL; device microbuilder:SOLDERJUMPER_2WAY0603 -> SparkFun-Passives:JUMPER-PAD-3-2OF3_NC_BY_TRACE_SMALL
Connections:
- net GND: now also S1.2, USB.GND; no longer S1.1, USB.GND@1
- net N$1: no longer S1.2
- net PB5: now also S1.1
Changed lines of the file:
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@@
 <?xml version="1.0" encoding="utf-8"?>
 <!DOCTYPE eagle SYSTEM "eagle.dtd">
-<eagle version="7.1.0">
+<eagle version="7.2.0">
 <drawing>
 <settings>
@@
 <layer number="54" name="bGND_GNDA" color="1" fill="9" visible="no" active="no"/>
 <layer number="56" name="wert" color="7" fill="1" visible="no" active="no"/>
+<layer number="57" name="tCAD" color="7" fill="1" visible="no" active="no"/>
 <layer number="90" name="Modules" color="5" fill="1" visible="yes" active="yes"/>
 <layer number="91" name="Nets" color="2" fill="1" visible="yes" active="yes"/>
@@
 <layer number="97" name="Info" color="7" fill="1" visible="yes" active="yes"/>
 <layer number="98" name="Guide" color="6" fill="1" visible="yes" active="yes"/>
+<layer number="99" name="SpiceOrder" color="7" fill="1" visible="yes" active="yes"/>
 <layer number="100" name="DocFrame" color="15" fill="1" visible="yes" active="yes"/>
 <layer number="101" name="Patch_Top" color="12" fill="4" visible="no" active="yes"/>
@@
 <layer number="111" name="MPL" color="7" fill="1" visible="yes" active="yes"/>
 <layer number="112" name="tSilk" color="7" fill="1" visible="yes" active="yes"/>
+<layer number="113" name="IDFDebug" color="7" fill="1" visible="yes" active="yes"/>
 <layer number="116" name="Patch_BOT" color="9" fill="4" visible="no" active="yes"/>
 <layer number="118" name="Rect_Pads" color="7" fill="1" visible="no" active="no"/>
@@
 <layer number="132" name="bAdjust" color="7" fill="1" visible="no" active="yes"/>
 <layer number="144" name="Drill_legend" color="7" fill="1" visible="no" active="yes"/>
+<layer number="150" name="Notes" color="7" fill="1" visible="yes" active="yes"/>
 <layer number="151" name="HeatSink" color="7" fill="1" visible="no" active="yes"/>
 <layer number="152" name="_bDocu" color="7" fill="1" visible="yes" active="yes"/>
+<layer number="153" name="FabDoc1" color="7" fill="1" visible="yes" active="yes"/>
+<layer number="154" name="FabDoc2" color="7" fill="1" visible="yes" active="yes"/>
+<layer number="155" name="FabDoc3" color="7" fill="1" visible="yes" active="yes"/>
 <layer number="199" name="Contour" color="7" fill="1" visible="yes" active="yes"/>
 <layer number="200" name="200bmp" color="1" fill="10" visible="no" active="yes"/>
@@
 <layer number="223" name="223bmp" color="24" fill="1" visible="no" active="no"/>
 <layer number="224" name="224bmp" color="25" fill="1" visible="no" active="no"/>
+<layer number="225" name="225bmp" color="7" fill="1" visible="yes" active="yes"/>
+<layer number="226" name="226bmp" color="7" fill="1" visible="yes" active="yes"/>
+<layer number="227" name="227bmp" color="7" fill="1" visible="yes" active="yes"/>
+<layer number="228" name="228bmp" color="7" fill="1" visible="yes" active="yes"/>
+<layer number="229" name="229bmp" color="7" fill="1" visible="yes" active="yes"/>
+<layer number="230" name="230bmp" color="7" fill="1" visible="yes" active="yes"/>
 <layer number="231" name="Eagle3D_PG1" color="7" fill="1" visible="yes" active="yes"/>
 <layer number="232" name="Eagle3D_PG2" color="7" fill="1" visible="yes" active="yes"/>
@@
 <part name="GND5" library="ATtami" deviceset="GND" device=""/>
 <part name="D5" library="ATtami" deviceset="SCHOTTKY-DIODE" device="SOD-323" value="Schottky"/>
-<part name="SJ1" library="ATtami" deviceset="SOLDERJUMPER" device="CLOSED"/>
+<part name="SJ1" library="SparkFun-Passives" deviceset="JUMPER-PAD-2-NC_BY_TRACE" device=""/>
 <part name="COIN_CELL_(+)" library="ATtami" deviceset="PINHD-1X1" device=""/>
 <part name="COIN_CELL_(-)" library="ATtami" deviceset="PINHD-1X1" device=""/>
 <part name="U2" library="ATtami" deviceset="ATTINY85-20SU" device=""/>
-<part name="1117" library="ATtami" deviceset="XXX1117" device="-SOT89"/>
-<part name="SJ2" library="microbuilder" deviceset="SOLDERJUMPER_2WAY" device="0603"/>
+<part name="1117" library="ATtami" deviceset="XXX1117" device=""/>
+<part name="SJ2" library="SparkFun-Passives" deviceset="JUMPER-PAD-3-2OF3_NC_BY_TRACE" device="_SMALL"/>
 </parts>
 <sheets>
@@
 <text x="59.944" y="144.272" size="1.778" layer="91">VCC (output)</text>
 <text x="23.114" y="126.492" size="1.778" layer="91">V_BAT (input)</text>
-<text x="204.978" y="94.996" size="1.778" layer="91" rot="R180">Reset</text>
-<text x="195.58" y="104.14" size="1.778" layer="91">midi jumper</text>
+<text x="212.344" y="103.378" size="1.778" layer="91" rot="R270">Reset</text>
+<text x="193.802" y="102.87" size="1.778" layer="91">midi jumper</text>
 </plain>
 <instances>
@@
 <instance part="D2" gate="LED" x="121.92" y="76.2"/>
 <instance part="GND16" gate="1" x="88.9" y="137.16"/>
-<instance part="GND13" gate="1" x="208.28" y="93.98"/>
+<instance part="GND13" gate="1" x="210.82" y="96.52"/>
 <instance part="GND1" gate="1" x="45.72" y="114.3"/>
 <instance part="GND6" gate="1" x="63.5" y="99.06" smashed="yes">
@@
 </instance>
 <instance part="U$1" gate="G$1" x="177.8" y="160.02"/>
-<instance part="S1" gate="G$1" x="198.12" y="96.52" smashed="yes" rot="R180"/>
+<instance part="S1" gate="G$1" x="210.82" y="106.68" smashed="yes" rot="R270"/>
 <instance part="USB" gate="G$1" x="53.34" y="86.36" smashed="yes">
 <attribute name="NAME" x="47.244" y="93.98" size="1.778" layer="95" ratio="10"/>
@@
 <attribute name="VALUE" x="108.712" y="147.828" size="1.27" layer="96" rot="R180"/>
 </instance>
-<instance part="SJ1" gate="1" x="134.62" y="96.52" rot="R180"/>
+<instance part="SJ1" gate="G$1" x="134.62" y="96.52" rot="R180"/>
 <instance part="COIN_CELL_(+)" gate="G$1" x="121.92" y="149.86" smashed="yes">
 <attribute name="NAME" x="124.46" y="149.479" size="1.778" layer="95"/>
@@
 </instance>
 <instance part="1117" gate="1" x="86.36" y="58.42" rot="R180"/>
-<instance part="SJ2" gate="G$1" x="193.04" y="106.68" smashed="yes" rot="R180">
-<attribute name="VALUE" x="198.12" y="113.03" size="1.778" layer="96" rot="R180"/>
-</instance>
+<instance part="SJ2" gate="G$1" x="193.04" y="106.68" smashed="yes" rot="R90"/>
 </instances>
 <busses>
@@
 <junction x="88.9" y="142.24"/>
 <pinref part="COIN_CELL_(-)" gate="G$1" pin="1"/>
-</segment>
-<segment>
-<pinref part="GND13" gate="1" pin="GND"/>
-<pinref part="S1" gate="G$1" pin="1"/>
-<wire x1="203.2" y1="96.52" x2="208.28" y2="96.52" width="0.1524" layer="91"/>
 </segment>
 <segment>
@@
 <pinref part="1117" gate="1" pin="GND"/>
 <wire x1="86.36" y1="101.6" x2="86.36" y2="66.04" width="0.1524" layer="91"/>
+<junction x="86.36" y="101.6"/>
 </segment>
 <segment>
@@
 </segment>
 <segment>
-<pinref part="GND4" gate="1" pin="GND"/>
-<pinref part="USB" gate="G$1" pin="GND@1"/>
-<wire x1="63.5" y1="81.28" x2="63.5" y2="78.74" width="0.1524" layer="91"/>
-</segment>
-<segment>
 <pinref part="J1" gate="A" pin="1"/>
 <wire x1="231.14" y1="129.54" x2="223.52" y2="129.54" width="0.1524" layer="91"/>
@@
 </segment>
 <segment>
-<pinref part="SJ1" gate="1" pin="1"/>
+<pinref part="SJ1" gate="G$1" pin="1"/>
 <pinref part="GND12" gate="1" pin="GND"/>
 <wire x1="139.7" y1="96.52" x2="142.24" y2="96.52" width="0.1524" layer="91"/>
+</segment>
+<segment>
+<pinref part="S1" gate="G$1" pin="2"/>
+<pinref part="GND13" gate="1" pin="GND"/>
+<wire x1="210.82" y1="101.6" x2="210.82" y2="99.06" width="0.2032" layer="91"/>
+</segment>
+<segment>
+<pinref part="USB" gate="G$1" pin="GND"/>
+<pinref part="GND4" gate="1" pin="GND"/>
+<wire x1="63.5" y1="81.28" x2="63.5" y2="78.74" width="0.1524" layer="91"/>
 </segment>
 </net>
@@
 <net name="PB4" class="0">
 <segment>
-<wire x1="182.88" y1="116.84" x2="190.5" y2="116.84" width="0.1524" layer="91"/>
 <pinref part="J1" gate="A" pin="6"/>
 <pinref part="U2" gate="A" pin="PB4"/>
+<wire x1="182.88" y1="116.84" x2="198.12" y2="116.84" width="0.1524" layer="91"/>
 <pinref part="SJ2" gate="G$1" pin="3"/>
-<wire x1="190.5" y1="116.84" x2="231.14" y2="116.84" width="0.1524" layer="91"/>
-<wire x1="190.5" y1="106.68" x2="190.5" y2="116.84" width="0.1524" layer="91"/>
-<junction x="190.5" y="116.84"/>
+<wire x1="198.12" y1="116.84" x2="231.14" y2="116.84" width="0.1524" layer="91"/>
+<wire x1="198.12" y1="116.84" x2="198.12" y2="106.68" width="0.1524" layer="91"/>
+<junction x="198.12" y="116.84"/>
 </segment>
 </net>
@@
 <segment>
 <pinref part="J1" gate="A" pin="7"/>
-<wire x1="231.14" y1="114.3" x2="195.58" y2="114.3" width="0.1524" layer="91"/>
 <pinref part="U2" gate="A" pin="PB5"/>
-<wire x1="182.88" y1="114.3" x2="195.58" y2="114.3" width="0.1524" layer="91"/>
+<wire x1="231.14" y1="114.3" x2="210.82" y2="114.3" width="0.1524" layer="91"/>
+<wire x1="210.82" y1="114.3" x2="187.96" y2="114.3" width="0.1524" layer="91"/>
+<wire x1="187.96" y1="114.3" x2="182.88" y2="114.3" width="0.1524" layer="91"/>
 <pinref part="SJ2" gate="G$1" pin="1"/>
-<wire x1="195.58" y1="114.3" x2="195.58" y2="106.68" width="0.1524" layer="91"/>
-<junction x="195.58" y="114.3"/>
+<wire x1="187.96" y1="106.68" x2="187.96" y2="114.3" width="0.1524" layer="91"/>
+<junction x="187.96" y="114.3"/>
+<pinref part="S1" gate="G$1" pin="1"/>
+<wire x1="210.82" y1="111.76" x2="210.82" y2="114.3" width="0.1524" layer="91"/>
+<junction x="210.82" y="114.3"/>
 </segment>
 </net>
@@
 <segment>
 <pinref part="D4" gate="LED" pin="C"/>
-<pinref part="SJ1" gate="1" pin="2"/>
+<pinref part="SJ1" gate="G$1" pin="2"/>
 <wire x1="129.54" y1="101.6" x2="129.54" y2="96.52" width="0.1524" layer="91"/>
 </segment>
@@
 <pinref part="R4" gate="G$1" pin="2"/>
 <wire x1="160.02" y1="86.36" x2="193.04" y2="86.36" width="0.1524" layer="91"/>
-<wire x1="193.04" y1="86.36" x2="193.04" y2="96.52" width="0.1524" layer="91"/>
 <pinref part="SJ2" gate="G$1" pin="2"/>
-<pinref part="S1" gate="G$1" pin="2"/>
-<wire x1="193.04" y1="96.52" x2="193.04" y2="104.14" width="0.1524" layer="91"/>
-<junction x="193.04" y="96.52"/>
-</segment>
-</net>
+<wire x1="193.04" y1="86.36" x2="193.04" y2="101.6" width="0.2032" layer="91"/>
+</segment>
+</net>

Commit message: Added remarks
Parts:
- removed 1117: (no value), ATtami:XXX1117
- added U3: 1117, ATtami:XXX1117
Connections:
- net GND: now also U3.GND; no longer 1117.GND
- net VCC: now also U3.OUT; no longer 1117.OUT
- net V_BAT: now also U3.IN; no longer 1117.IN
Other:
- note added: "* See Note 1"
- note added: "Notes: 1. Assemble either U1 or U3. (!!! never both of them !!!) 2. Cut jumper SJ1 in order to save battery energy. 3. Switch possition of midi jumper and dissable the RESET function in order to use PB5 as DP USB signal. 4. D1 and D2 are Blue LEDs their forward voltage is 3.2V. They might not light when using coin cell or low Vi_BAT. 5. When VCC is less than 5V the system clock of the ATTINY85 sh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"
- note removed: "Notes: 1. D1 and D2 are Blue LEDs they might not light when using Vi_BAT <4V~ 2. When VCC is less than 5V change the system clock of the ATTINY85 to 8MHz or less (refer to the datasheet P163 Section 21-3 Speed)"
- moved on the sheet: C1, C2, COIN_CELL_(+), COIN_CELL_(-), D1, D2, D3, D4, D5, J1, J2, J3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
