File: shields/ATTAMI-Shield-template.brd (EAGLE design)
At the start: 22.8 x 22.9 mm, 6 parts

Commit message: updated shield tamplete to only use ATtami lib parts
Parts:
- J1: device microbuilder:1X07_ROUND -> ATtami:1X07_ROUND
- J2, J3: device microbuilder:1X02_ROUND -> ATtami:1X02_ROUND
- U$1, U$2: device microbuilder:MOUNTINGHOLE_2.0_PLATED -> ATtami:MOUNTINGHOLE_2.0_PLATED
Changed lines of the file:
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@@
 </autorouter>
 <elements>
-<element name="U$1" library="microbuilder" package="MOUNTINGHOLE_2.0_PLATED" value="MOUNTINGHOLE2.0" x="2.54" y="20.32" smashed="yes" rot="R270"/>
-<element name="U$2" library="microbuilder" package="MOUNTINGHOLE_2.0_PLATED" value="MOUNTINGHOLE2.0" x="20.32" y="20.32" smashed="yes"/>
-<element name="J2" library="microbuilder" package="1X02_ROUND" value="" x="21.59" y="12.7" smashed="yes" rot="R270">
+<element name="U$1" library="ATtami" package="MOUNTINGHOLE_2.0_PLATED" value="MOUNTINGHOLE2.0" x="2.54" y="20.32" smashed="yes" rot="R270"/>
+<element name="U$2" library="ATtami" package="MOUNTINGHOLE_2.0_PLATED" value="MOUNTINGHOLE2.0" x="20.32" y="20.32" smashed="yes"/>
+<element name="J2" library="ATtami" package="1X02_ROUND" value="" x="21.59" y="12.7" smashed="yes" rot="R270">
 <attribute name="NAME" x="20.843240625" y="8.666478125" size="1.27" layer="37" ratio="10"/>
 </element>
-<element name="J3" library="microbuilder" package="1X02_ROUND" value="" x="21.59" y="2.54" smashed="yes" rot="R270">
+<element name="J3" library="ATtami" package="1X02_ROUND" value="" x="21.59" y="2.54" smashed="yes" rot="R270">
 <attribute name="NAME" x="20.77211875" y="5.6286375" size="1.27" layer="37" ratio="10"/>
 </element>
-<element name="J1" library="microbuilder" package="1X07_ROUND" value="" x="1.27" y="8.89" smashed="yes" rot="R270">
+<element name="J1" library="ATtami" package="1X07_ROUND" value="" x="1.27" y="8.89" smashed="yes" rot="R270">
 <attribute name="VALUE" x="-1.905" y="17.78" size="0.4064" layer="27" ratio="10" rot="R270"/>
 </element>
