File: shields/tutuShield/tutuShield.brd (EAGLE design)
At the start: 22.8 x 22.9 mm, 19 parts, among them IC1 IC_MSGEQ7-SOIC8

Commit message: fixed tutushield, needs review
Routing:
- net PB3: track 10.8 -> 21.6 mm
- net PB1: track 20.3 -> 9.88 mm, vias 2 -> 0
Changed lines of the file:
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@@
 <?xml version="1.0" encoding="utf-8"?>
 <!DOCTYPE eagle SYSTEM "eagle.dtd">
-<eagle version="7.1.0">
+<eagle version="7.2.0">
 <drawing>
 <settings>
@@
 <layer number="20" name="Dimension" color="15" fill="1" visible="yes" active="yes"/>
 <layer number="21" name="tPlace" color="16" fill="1" visible="yes" active="yes"/>
-<layer number="22" name="bPlace" color="14" fill="1" visible="yes" active="yes"/>
+<layer number="22" name="bPlace" color="14" fill="1" visible="no" active="yes"/>
 <layer number="23" name="tOrigins" color="15" fill="1" visible="yes" active="yes"/>
 <layer number="24" name="bOrigins" color="15" fill="1" visible="yes" active="yes"/>
@@
 <contactref element="Q1-3" pad="2"/>
 <contactref element="Q2" pad="2"/>
-<wire x1="17.907" y1="8.139" x2="21.59" y2="11.43" width="0" layer="19" extent="1-1"/>
-<wire x1="21.59" y1="6.477" x2="17.907" y2="8.139" width="0" layer="19" extent="1-1"/>
-<wire x1="21.59" y1="1.27" x2="21.59" y2="6.477" width="0" layer="19" extent="1-1"/>
-<wire x1="13.705" y1="2.921" x2="15.378" y2="1.016" width="0" layer="19" extent="1-1"/>
 <wire x1="1.27" y1="16.51" x2="5.08" y2="16.51" width="0.3048" layer="1"/>
 <wire x1="5.08" y1="16.51" x2="5.08" y2="17.272" width="0.3048" layer="1"/>
@@
 <signal name="PB1">
 <contactref element="J1" pad="3"/>
-<wire x1="16.51" y1="9.525" x2="17.018" y2="10.16" width="0.254" layer="1"/>
-<wire x1="17.018" y1="10.16" x2="17.018" y2="11.811" width="0.254" layer="1"/>
-<wire x1="17.018" y1="11.811" x2="9.398" y2="11.811" width="0.254" layer="1"/>
-<wire x1="9.398" y1="11.811" x2="8.509" y2="11.176" width="0.254" layer="1"/>
-<wire x1="8.509" y1="11.176" x2="7.874" y2="9.525" width="0.254" layer="1"/>
-<via x="7.874" y="9.525" extent="1-16" drill="0.6" shape="square"/>
-<wire x1="7.874" y1="9.525" x2="7.239" y2="9.525" width="0.254" layer="16"/>
-<wire x1="7.239" y1="9.525" x2="5.334" y2="11.43" width="0.254" layer="16"/>
-<via x="5.334" y="11.43" extent="1-16" drill="0.6" shape="square"/>
-<wire x1="5.334" y1="11.43" x2="1.27" y2="11.43" width="0.254" layer="1"/>
 <contactref element="R2" pad="2"/>
-<wire x1="9.398" y1="11.811" x2="10.414" y2="13.197" width="0" layer="19" extent="1-1"/>
+<wire x1="1.27" y1="11.43" x2="7.62" y2="11.43" width="0.4064" layer="1"/>
+<wire x1="7.62" y1="11.43" x2="9.271" y2="13.081" width="0.4064" layer="1"/>
+<wire x1="9.271" y1="13.081" x2="10.298" y2="13.081" width="0.4064" layer="1"/>
+<wire x1="10.298" y1="13.081" x2="10.414" y2="13.197" width="0.4064" layer="1"/>
 </signal>
 <signal name="PB2">
@@
 <signal name="PB3">
 <contactref element="J1" pad="5"/>
-<wire x1="1.27" y1="6.35" x2="3.302" y2="6.35" width="0.254" layer="1"/>
-<wire x1="3.302" y1="6.35" x2="8.89" y2="12.446" width="0.254" layer="1"/>
-<wire x1="8.89" y1="12.446" x2="9.409" y2="12.446" width="0.254" layer="1"/>
 <contactref element="IC1" pad="7"/>
-<wire x1="9.409" y1="12.446" x2="15.427" y2="9.525" width="0" layer="19" extent="1-1"/>
+<wire x1="15.427" y1="9.525" x2="16.383" y2="9.525" width="0.254" layer="1"/>
+<wire x1="16.383" y1="9.525" x2="17.145" y2="10.287" width="0.254" layer="1"/>
+<wire x1="17.145" y1="10.287" x2="17.145" y2="11.43" width="0.254" layer="1"/>
+<wire x1="17.145" y1="11.43" x2="16.891" y2="11.684" width="0.254" layer="1"/>
+<wire x1="16.891" y1="11.684" x2="9.017" y2="11.684" width="0.254" layer="1"/>
+<wire x1="9.017" y1="11.684" x2="3.429" y2="6.096" width="0.254" layer="1"/>
+<wire x1="3.429" y1="6.096" x2="1.524" y2="6.096" width="0.254" layer="1"/>
+<wire x1="1.524" y1="6.096" x2="1.27" y2="6.35" width="0.254" layer="1"/>
 </signal>
 <signal name="PB4">
@@
 <contactref element="C1" pad="1"/>
 <contactref element="R1" pad="1"/>
-<wire x1="12.7" y1="3.937" x2="13.208" y2="3.937" width="0" layer="19" extent="1-16"/>
 <wire x1="13.208" y1="3.937" x2="15.367" y2="3.937" width="0.3048" layer="1"/>
 <wire x1="15.367" y1="3.937" x2="15.367" y2="3.048" width="0.3048" layer="1"/>
