File: kicad/attami.sch (KiCad schematic (older format))
At the start: 19 parts

Commit message: added project kicad extension
Parts:
- removed U?: AP111750, TO_SOT_Packages_SMD:SOT-223, symbol AP111750
- added U1: AP111750, TO_SOT_Packages_SMD:SOT-223, symbol AP111750
- C1, C2: renamed from C?; footprint (none) -> Capacitors_SMD:C_0805
- D1, D3, D4: renamed from D?; footprint (none) -> LEDs:LED_0805
- D2: renamed from D?; footprint (none) -> Diodes_SMD:SOD-323
- IC1: renamed from IC?; footprint SO8-200 -> SMD_Packages:SOIC-8-N
- JP1: renamed from JP?; footprint (none) -> Connect:GS2
- JP2: renamed from JP?; footprint (none) -> Connect:GS3
- P1, P3: renamed from P?; footprint (none) -> Pin_Headers:Pin_Header_Straight_1x02
- P2: renamed from P?; footprint (none) -> Connect:USB_Mini-B
- P4: renamed from P?; footprint (none) -> Pin_Headers:Pin_Header_Straight_1x07
- R1, R2, R3, R4: renamed from R?; footprint (none) -> Resistors_SMD:R_0805
- SW1: renamed from SW?; footprint (none) -> Buttons_Switches_SMD:SW_SPST_EVQPE1
Connections:
- net GND: now also U1.1 (GND/ADJ)
- net VCC: now also C2.1, D2.1 (K), IC1.8 (VCC), R1.2, R2.2, U1.2 (VO), U1.4 (VO)
- net V_BAT: now also U1.3 (VI)
- no-connect marks 0 -> 2
Other:
- moved on the sheet: C1, C2, D1, D2, D3, D4, IC1, JP1, JP2, P1, P2, P3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
